File: pcb/extrava/extrava.kicad_sch (KiCad schematic)
At the start: 24 parts, among them J1 Conn_01x01_Socket, J2 Conn_01x01_Socket, J3 Conn_01x01_Socket, J4 Conn_01x01_Socket, U1 XIAO_ESP32C3, U2 AD5941BCPZ, Y1 ABM8-16.000MHZ-10-1-U-T

Commit message: fix(layout): closer decoupling caps
Parts:
- J1, J2, J3, J4: footprint Connector_Wire:SolderWire-0.75sqmm_1x01_D1.25mm_OD3.5mm_Relief -> Connector_Wire:SolderWire-0.75sqmm_1x01_D1.25mm_OD3.5mm
Other:
- note added: "AFE (Analog Front End)"
- note removed: "AFE"
Changed lines of the file:
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@@
 		)
 	)
-	(text "AFE"
+	(text "AFE (Analog Front End)"
 		(exclude_from_sim no)
-		(at 162.814 61.976 0)
+		(at 209.804 62.484 0)
 		(effects
 			(font
@@
 			)
 		)
-		(property "Footprint" "Connector_Wire:SolderWire-0.75sqmm_1x01_D1.25mm_OD3.5mm_Relief"
+		(property "Footprint" "Connector_Wire:SolderWire-0.75sqmm_1x01_D1.25mm_OD3.5mm"
 			(at 107.95 167.64 0)
 			(effects
@@
 			)
 		)
-		(property "Footprint" "Connector_Wire:SolderWire-0.75sqmm_1x01_D1.25mm_OD3.5mm_Relief"
+		(property "Footprint" "Connector_Wire:SolderWire-0.75sqmm_1x01_D1.25mm_OD3.5mm"
 			(at 107.95 162.56 0)
 			(effects
@@
 			)
 		)
-		(property "Footprint" "Connector_Wire:SolderWire-0.75sqmm_1x01_D1.25mm_OD3.5mm_Relief"
+		(property "Footprint" "Connector_Wire:SolderWire-0.75sqmm_1x01_D1.25mm_OD3.5mm"
 			(at 107.95 160.02 0)
 			(effects
@@
 			)
 		)
-		(property "Footprint" "Connector_Wire:SolderWire-0.75sqmm_1x01_D1.25mm_OD3.5mm_Relief"
+		(property "Footprint" "Connector_Wire:SolderWire-0.75sqmm_1x01_D1.25mm_OD3.5mm"
 			(at 107.95 165.1 0)
 			(effects
